File: pcbs/combined.kicad_pcb (KiCad board)
At the start: 2 copper layers, 267.6 x 86.8 mm, 96 parts

Commit message: move right pads of pg1316s footprint to the center to enable better solder joints
Parts:
- CPG1316 (x42): footprint CPG1316S01D02_mikeholscher -> pg1316sexportfootprint:CPG1316S01D02_mikeholscher
Other:
- outline, holes or cut-outs redrawn

Commit message: rerouted switch footprints after chaning the footprint to account for a smaller pad distance
Parts:
- moved JST1 0.06 mm to (236.3, 60.8)
Other:
- outline, holes or cut-outs redrawn

Commit message: updated gerbers for small changes in the pcb
Routing:
- net P0: track 305.1 -> 301.6 mm
- net RAW: track 119.2 -> 120.1 mm
Other:
- outline, holes or cut-outs redrawn

Commit message: minor tweaks to the pcb files => also changes in the gerbers. making some last adjustments before ordering
Routing:
- net RST: track 206.2 -> 207.2 mm

Commit message: Changes to the pcb: added small mounting holes
Parts:
- added REF**: TestPoint_Plated_Hole_D2.0mm, TestPoint:TestPoint_Plated_Hole_D2.0mm, F.Cu at (296.9, 36.4)
- added REF**: TestPoint_Plated_Hole_D2.0mm, TestPoint:TestPoint_Plated_Hole_D2.0mm, F.Cu at (140.1, 36.4)
- added REF**: TestPoint_Plated_Hole_D2.0mm, TestPoint:TestPoint_Plated_Hole_D2.0mm, F.Cu at (151.1, 93.7)
- added REF**: TestPoint_Plated_Hole_D2.0mm, TestPoint:TestPoint_Plated_Hole_D2.0mm, F.Cu at (285.9, 93.7)
- added mouse-bite-1mm-3mm: VAL**, mouse-bite:mouse-bite-1mm-3mm, F.Cu at (218.6, 44.5)
- added mouse-bite-1mm-3mm: VAL**, mouse-bite:mouse-bite-1mm-3mm, F.Cu at (218.6, 98.1)
- added mouse-bite-1mm-3mm: VAL**, mouse-bite:mouse-bite-1mm-3mm, F.Cu at (218.6, 96.8)
- added mouse-bite-1mm-3mm: VAL**, mouse-bite:mouse-bite-1mm-3mm, F.Cu at (218.6, 42.0)
- moved mouse-bite-1mm-3mm 2.35 mm to (218.6, 99.3)
- moved mouse-bite-1mm-3mm 1.05 mm to (218.5, 43.3)
Routing:
- net GND: track 248.3 -> 250.0 mm
- net RST: track 207.2 -> 208.8 mm
Other:
- outline, holes or cut-outs redrawn

Commit message: moved left pad of pg1316s footprint to the middle by 1mm to improve connection + align more closely to the actual pads of the switch, updated custom footprint file, updated footprints in kicad + rerouted
Routing:
- net P4: track 340.9 -> 336.8 mm
- net P8: track 290.3 -> 293.7 mm
- net P7: track 282.4 -> 285.7 mm
- net P9: track 317.4 -> 319.9 mm
- net P6: track 288.3 -> 290.6 mm
- net P2: track 343.8 -> 345.8 mm
- net P3: track 280.6 -> 279.5 mm

Commit message: small updates to the pcb
Routing:
- net P3: track 279.5 -> 280.9 mm

Commit message: tweaks to the pcb
Parts:
- added REF**: TestPoint_Plated_Hole_D2.0mm, TestPoint:TestPoint_Plated_Hole_D2.0mm, F.Cu at (301.4, 95.5)
- added REF**: TestPoint_Plated_Hole_D2.0mm, TestPoint:TestPoint_Plated_Hole_D2.0mm, F.Cu at (135.5, 95.6)
- added REF**: TestPoint_Plated_Hole_D2.0mm, TestPoint:TestPoint_Plated_Hole_D2.0mm, F.Cu at (223.6, 97.2)
- added REF**: TestPoint_Plated_Hole_D2.0mm, TestPoint:TestPoint_Plated_Hole_D2.0mm, F.Cu at (213.4, 97.2)
