File: pcbs/reversible.kicad_pcb (KiCad board)
At the start: 2 copper layers, 132.7 x 86.8 mm, 50 parts

Commit message: more tweaks to to the pcb
Parts:
- moved JST1 0.21 mm to (200.8, 60.9)
Routing:
- net P9: track 154.1 -> 148.5 mm
- net RAW: track 105.1 -> 101.4 mm
- net P8: track 127.5 -> 124.0 mm
- net P3: track 164.8 -> 168.2 mm
- net P5: track 170.0 -> 166.9 mm
- net P2: track 201.1 -> 198.9 mm
- net P4: track 184.3 -> 182.7 mm
- net P0: track 174.6 -> 175.3 mm
- net P10: track 18.3 -> 19.0 mm
- net RST: track 96.7 -> 96.1 mm

Commit message: more changes to the pcb
Routing:
- net VCC5: track 22.5 -> 21.4 mm

Commit message: minor changes to the routing
Routing:
- net P3: track 168.2 -> 167.2 mm
