File: pcbs/reversible.kicad_pcb (KiCad board)
At the start: 2 copper layers, 132.7 x 86.8 mm, 50 parts

Commit message: cosmetic changes
Routing:
- net BAT_P: track 70.5 -> 108.8 mm, vias 2 -> 3
- net RAW: track 103.9 -> 91.3 mm
- net P2: track 200.3 -> 206.3 mm
- net P9: track 150.9 -> 148.5 mm
- net GND: track 179.2 -> 178.0 mm, vias 1 -> 5
Other:
- board text added: "chalk@v0.1.1"
- board text removed: "chalk@v0.1"

Commit message: small cosmetic changes to the routing
Routing:
- net P0: track 173.6 -> 168.9 mm
- net P2: track 206.3 -> 203.2 mm
- net RAW: track 91.3 -> 88.6 mm
- net P7: track 151.6 -> 148.9 mm
- net GND: track 178.0 -> 176.0 mm
- net P1: track 185.3 -> 183.6 mm
- net P3: track 168.5 -> 167.1 mm
- net RST: track 96.6 -> 95.4 mm
- net inner_top: track 8.45 -> 7.60 mm
- net VCC33: track 20.0 -> 19.1 mm
- net P9: track 148.5 -> 147.6 mm
- net P8: track 125.8 -> 125.0 mm
- net VCC5: track 20.9 -> 20.1 mm
- net P6: track 141.3 -> 140.6 mm
- net middle_top: track 8.24 -> 7.60 mm
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
Commit message: cosmetic changes to the pcb
Routing:
- net GND: track 176.0 -> 169.5 mm, vias 5 -> 49
- net BAT_P: track 108.4 -> 109.6 mm
- net P1: track 183.6 -> 184.2 mm
- added copper zone on B.Cu, net GND
- added copper zone on F.Cu, net GND
- removed copper zone on B.Cu, net (none)
- removed copper zone on F.Cu, net (none)
Other:
- board text added: "chalk@v0.1.2"
- board text removed: "chalk@v0.1.1"
